Commit message: Added display.launch to view and test model in rviz. Added geometry tag to rail.xacro base link visual.

File: src/rail_description/urdf/rail.xacro (robot description, xacro)
@@ -14,5 +14,7 @@
     </collision>
     <visual>
-        <box size="1 1 0.5"/>
+        <geometry>
+            <box size="1 1 0.5"/>
+        </geometry>
     </visual>
     <inertial>

Commit message: moved base up

File: src/rail_description/urdf/rail.xacro (robot description, xacro)
@@ -4,4 +4,5 @@
 <link name="world"/>
 <joint name="world_fixed" type="fixed">
+    <origin xyz="0 0 0.5" rpy="0 0 0"/>
     <parent link="world"/>
     <child link="base"/>

Commit message: Added first moveable link yaw

File: src/rail_description/urdf/rail.xacro (robot description, xacro)
@@ -4,5 +4,5 @@
 <link name="world"/>
 <joint name="world_fixed" type="fixed">
-    <origin xyz="0 0 0.5" rpy="0 0 0"/>
+    <origin xyz="0 0 0.25" rpy="0 0 0"/>
     <parent link="world"/>
     <child link="base"/>
@@ -27,3 +27,28 @@
     </inertial>
 </link>
+<joint name="yaw" type="continuous">
+    <parent link="base"/>
+    <child link="vertical_strut"/>
+    <origin xyz="0 0 1.25" rpy="0 0 0"/>
+    <axis xyz="0 0 1"/>
+</joint>
+<link name="vertical_strut">
+    <collision>
+        <geometry>
+            <box size="0.5 0.5 2"/>
+        </geometry>
+    </collision>
+    <visual>
+        <geometry>
+            <box size="0.5 0.5 2"/>
+        </geometry>
+    </visual>
+    <inertial>
+        <mass value="10.0"/>
+        <inertia
+	    ixx="${10 / 12.0 * (0.5 + 2*2)}" ixy="0.0" ixz="0.0"
+	    iyy="${10 / 12.0 * (2*2 + 0.5)}" iyz="0.0"
+	    izz="${10 / 12.0 * (0.5 + 0.5)}"/>
+    </inertial>
+</link>
 </robot>

Commit message: Added second joint pitch

File: src/rail_description/urdf/rail.xacro (robot description, xacro)
@@ -52,3 +52,31 @@
     </inertial>
 </link>
+<joint name="pitch" type="continuous">
+    <parent link="vertical_strut"/>
+    <child link="barrel"/>
+    <origin xyz="0 0.5 0.75" rpy="0 0 0"/>
+    <axis xyz="0 1 0"/>
+</joint>
+<link name="barrel">
+    <collision>
+        <origin xyz="0.75 0 0" rpy="0 ${(PI)/2} 0"/>
+        <geometry>
+            <box size="0.5 0.5 2"/>
+        </geometry>
+    </collision>
+    <visual>
+        <origin xyz="0.75 0 0" rpy="0 ${(PI)/2} 0"/>
+        <geometry>
+            <box size="0.5 0.5 2"/>
+        </geometry>
+    </visual>
+    <inertial>
+        <origin xyz="0.75 0 0" rpy="0 ${(PI)/2} 0"/>
+        <mass value="10.0"/>
+        <inertia
+	    ixx="${10 / 12.0 * (0.5 + 2*2)}" ixy="0.0" ixz="0.0"
+	    iyy="${10 / 12.0 * (2*2 + 0.5)}" iyz="0.0"
+	    izz="${10 / 12.0 * (0.5 + 0.5)}"/>
+    </inertial>
+</link>
 </robot>

Commit message: Added transmission tags and gazebo support

File: src/rail_description/urdf/rail.xacro (robot description, xacro)
@@ -2,4 +2,18 @@
 <robot name="rail" xmlns:xacro="http://www.ros.org/wiki/xacro">
 <xacro:property name="PI" value="3.1415926535897931"/>
+<gazebo>
+    <plugin name="gazebo_ros_control" filename="libgazebo_ros_control.so">
+      <robotNamespace>/rail</robotNamespace>
+      <robotSimType>gazebo_ros_control/DefaultRobotHWSim</robotSimType>
+    </plugin>
+</gazebo>
+<gazebo reference="vertical_strut">
+    <mu1>0.2</mu1>
+    <mu2>0.2</mu2>
+</gazebo>
+<gazebo reference="barrel">
+    <mu1>0.2</mu1>
+    <mu2>0.2</mu2>
+</gazebo>
 <link name="world"/>
 <joint name="world_fixed" type="fixed">
@@ -80,3 +94,23 @@
     </inertial>
 </link>
+<transmission name="yaw_transmission">
+    <type>transmission_interface/SimpleTransmission</type>
+    <joint name="yaw">
+      <hardwareInterface>hardware_interface/EffortJointInterface</hardwareInterface>
+    </joint>
+    <actuator name="motor2">
+      <hardwareInterface>hardware_interface/EffortJointInterface</hardwareInterface>
+      <mechanicalReduction>1</mechanicalReduction>
+    </actuator>
+</transmission>
+<transmission name="pitch_transmission">
+    <type>transmission_interface/SimpleTransmission</type>
+    <joint name="pitch">
+      <hardwareInterface>hardware_interface/EffortJointInterface</hardwareInterface>
+    </joint>
+    <actuator name="motor2">
+      <hardwareInterface>hardware_interface/EffortJointInterface</hardwareInterface>
+      <mechanicalReduction>1</mechanicalReduction>
+    </actuator>
+</transmission>
 </robot>

Commit message: Corrected controller names in rail_control.launch and corrected inertial values in rail.xacro

File: src/rail_description/urdf/rail.xacro (robot description, xacro)
@@ -59,9 +59,9 @@
     </visual>
     <inertial>
-        <mass value="10.0"/>
+        <mass value="1.0"/>
         <inertia
-	    ixx="${10 / 12.0 * (0.5 + 2*2)}" ixy="0.0" ixz="0.0"
-	    iyy="${10 / 12.0 * (2*2 + 0.5)}" iyz="0.0"
-	    izz="${10 / 12.0 * (0.5 + 0.5)}"/>
+	    ixx="${1 / 12.0 * (0.5*0.5 + 2*2)}" ixy="0.0" ixz="0.0"
+	    iyy="${1 / 12.0 * (2*2 + 0.5*0.5)}" iyz="0.0"
+	    izz="${1 / 12.0 * (0.5*0.5 + 0.5*0.5)}"/>
     </inertial>
 </link>
@@ -87,9 +87,9 @@
     <inertial>
         <origin xyz="0.75 0 0" rpy="0 ${(PI)/2} 0"/>
-        <mass value="10.0"/>
+        <mass value="1.0"/>
         <inertia
-	    ixx="${10 / 12.0 * (0.5 + 2*2)}" ixy="0.0" ixz="0.0"
-	    iyy="${10 / 12.0 * (2*2 + 0.5)}" iyz="0.0"
-	    izz="${10 / 12.0 * (0.5 + 0.5)}"/>
+	    ixx="${1 / 12.0 * (0.5*0.5 + 2*2)}" ixy="0.0" ixz="0.0"
+	    iyy="${1 / 12.0 * (2*2 + 0.5*0.5)}" iyz="0.0"
+	    izz="${1 / 12.0 * (0.5*0.5 + 0.5*0.5)}"/>
     </inertial>
 </link>

Commit message: Modified ros_control aspects to improve control. Note: ros_control position/effort controller struggled with an unbalanced arm of this size. A temporary solution was reached by balancing the barrel, but that issue should be revisited later

File: src/rail_description/urdf/rail.xacro (robot description, xacro)
@@ -45,4 +45,5 @@
     <child link="vertical_strut"/>
     <origin xyz="0 0 1.25" rpy="0 0 0"/>
+    <limit effort="10000" velocity="10.0"/>
     <axis xyz="0 0 1"/>
 </joint>
@@ -70,9 +71,10 @@
     <child link="barrel"/>
     <origin xyz="0 0.5 0.75" rpy="0 0 0"/>
+    <limit effort="10000" velocity="10.0"/>
     <axis xyz="0 1 0"/>
 </joint>
 <link name="barrel">
     <collision>
-        <origin xyz="0.75 0 0" rpy="0 ${(PI)/2} 0"/>
+        <origin xyz="0 0 0" rpy="0 ${(PI)/2} 0"/>
         <geometry>
             <box size="0.5 0.5 2"/>
@@ -80,5 +82,5 @@
     </collision>
     <visual>
-        <origin xyz="0.75 0 0" rpy="0 ${(PI)/2} 0"/>
+        <origin xyz="0 0 0" rpy="0 ${(PI)/2} 0"/>
         <geometry>
             <box size="0.5 0.5 2"/>
@@ -86,10 +88,10 @@
     </visual>
     <inertial>
-        <origin xyz="0.75 0 0" rpy="0 ${(PI)/2} 0"/>
-        <mass value="1.0"/>
+        <origin xyz="0 0 0" rpy="0 ${(PI)/2} 0"/>
+        <mass value="0.5"/>
         <inertia
-	    ixx="${1 / 12.0 * (0.5*0.5 + 2*2)}" ixy="0.0" ixz="0.0"
-	    iyy="${1 / 12.0 * (2*2 + 0.5*0.5)}" iyz="0.0"
-	    izz="${1 / 12.0 * (0.5*0.5 + 0.5*0.5)}"/>
+	    ixx="${0.5 / 12.0 * (0.5*0.5 + 2*2)}" ixy="0.0" ixz="0.0"
+	    iyy="${0.5 / 12.0 * (2*2 + 0.5*0.5)}" iyz="0.0"
+	    izz="${0.5 / 12.0 * (0.5*0.5 + 0.5*0.5)}"/>
     </inertial>
 </link>

Commit message: modified third link name

File: src/rail_description/urdf/rail.xacro (robot description, xacro)
@@ -12,5 +12,5 @@
     <mu2>0.2</mu2>
 </gazebo>
-<gazebo reference="barrel">
+<gazebo reference="horizontal_strut">
     <mu1>0.2</mu1>
     <mu2>0.2</mu2>
@@ -69,10 +69,10 @@
 <joint name="pitch" type="continuous">
     <parent link="vertical_strut"/>
-    <child link="barrel"/>
+    <child link="horizontal_strut"/>
     <origin xyz="0 0.5 0.75" rpy="0 0 0"/>
     <limit effort="10000" velocity="10.0"/>
     <axis xyz="0 1 0"/>
 </joint>
-<link name="barrel">
+<link name="horizontal_strut">
     <collision>
         <origin xyz="0 0 0" rpy="0 ${(PI)/2} 0"/>

Commit message: Moved horizontal joint to unbalanced state

File: src/rail_description/urdf/rail.xacro (robot description, xacro)
@@ -76,5 +76,5 @@
 <link name="horizontal_strut">
     <collision>
-        <origin xyz="0 0 0" rpy="0 ${(PI)/2} 0"/>
+        <origin xyz="0.75 0 0" rpy="0 ${(PI)/2} 0"/>
         <geometry>
             <box size="0.5 0.5 2"/>
@@ -82,5 +82,5 @@
     </collision>
     <visual>
-        <origin xyz="0 0 0" rpy="0 ${(PI)/2} 0"/>
+        <origin xyz="0.75 0 0" rpy="0 ${(PI)/2} 0"/>
         <geometry>
             <box size="0.5 0.5 2"/>
@@ -88,5 +88,5 @@
     </visual>
     <inertial>
-        <origin xyz="0 0 0" rpy="0 ${(PI)/2} 0"/>
+        <origin xyz="0.75 0 0" rpy="0 ${(PI)/2} 0"/>
         <mass value="0.5"/>
         <inertia

Commit message: successful publishing of a std_msgs::Float64 message

File: src/rail_description/urdf/rail.xacro (robot description, xacro)
@@ -76,5 +76,5 @@
 <link name="barrel">
     <collision>
-        <origin xyz="0 0 0" rpy="0 ${(PI)/2} 0"/>
+        <origin xyz="0.75 0 0" rpy="0 ${(PI)/2} 0"/>
         <geometry>
             <box size="0.5 0.5 2"/>
@@ -82,5 +82,5 @@
     </collision>
     <visual>
-        <origin xyz="0 0 0" rpy="0 ${(PI)/2} 0"/>
+        <origin xyz="0.75 0 0" rpy="0 ${(PI)/2} 0"/>
         <geometry>
             <box size="0.5 0.5 2"/>
@@ -88,5 +88,5 @@
     </visual>
     <inertial>
-        <origin xyz="0 0 0" rpy="0 ${(PI)/2} 0"/>
+        <origin xyz="0.75 0 0" rpy="0 ${(PI)/2} 0"/>
         <mass value="0.5"/>
         <inertia
